Commit message: update

File: config/gazebo_arm_assembly.urdf (robot description, URDF)
Before this commit: robot arm_assembly, 10 links, 9 joints
Joints:
- joint joint_1: limit lower=-3.2 upper=-0.6 effort=300 velocity=3 -> lower=2.55 upper=5.7280 effort=300 velocity=3
- joint joint_2: limit lower=-0.2 upper=3.1 effort=200 velocity=3 -> lower=-0.35 upper=3.5340 effort=200 velocity=3
- joint joint_3: limit lower=0 upper=2.5549 effort=200 velocity=3 -> lower=-0.0488 upper=5.2280 effort=200 velocity=3
- joint joint_4: limit lower=-3.0 upper=3.0 effort=200 velocity=3 -> lower=-3.142 upper=3.142 effort=200 velocity=3
- joint joint_5: limit lower=-2.800 upper=0.61 effort=200 velocity=3 -> lower=-3.764 upper=0.6419 effort=200 velocity=3
- joint joint_6: limit lower=0 upper=6.284 effort=200 velocity=3 -> lower=-3.142 upper=3.142 effort=200 velocity=3
